File: classic/cls_car/pcb/slimarm_carambola/slimarm_carambola_nonand/slimarm_carambola.kicad_sch (KiCad schematic)
At the start: 72 parts, among them J1 USB_C_Receptacle_USB2.0, J2 Conn_01x05, J3 Conn_01x04, J4 Conn_01x04, U1 AT91SAM9G25-CU, U2 16bit-DDR2-8bank-FBGA84, U3 W25Q128JVS, U5 XC6206PxxxMR, U6 XC6206PxxxMR, U7 XC6206PxxxMR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

Commit message: fixed carambola board; board 3d models
Parts:
- removed C17, C18: 100nF, jlywxy:0402, symbol Device:C
- removed J2: Conn_01x05, Connector_PinHeader_2.00mm:PinHeader_1x05_P2.00mm_Vertical, symbol Connector_Generic:Conn_01x05
- removed J3, J4: Conn_01x04, Connector_PinHeader_2.00mm:PinHeader_1x04_P2.00mm_Vertical, symbol Connector_Generic:Conn_01x04
- removed R16, R17, R18, R19: 10k, jlywxy:0402, symbol Device:R
- removed R4: NC, jlywxy:0603, symbol Device:R
- removed R6: 0, jlywxy:0603, symbol Device:R
- removed R8: 1.5k, jlywxy:0603, symbol Device:R
- removed Y1: Crystal_GND24, jlywxy:Crystal_5032-4P, symbol Device:Crystal_GND24
- added C28: 100nF, jlywxy:0402, symbol Device:C
- added J2: Conn_01x04, Connector_PinHeader_2.54mm:PinHeader_1x04_P2.54mm_Vertical, symbol Connector_Generic:Conn_01x04
- added J4: DF13A-7P-1.25H21, jlywxy:DF13A-7P-1.25H21, symbol jlywxy:DF13A-7P-1.25H21
- added R13, R22, R23, R24: 10k, jlywxy:0402, symbol Device:R
- added SW1: SW_MEC_5E, jlywxy:BUTTON_4P_3x4, symbol Switch:SW_MEC_5E
- added U4: ~, jlywxy:MicroSD-TF_PUSH-SHOUHAN, symbol jlywxy:MicroSD-TF_PUSH-SHOUHAN
- added Y1: Crystal, Crystal:Crystal_SMD_5032-2Pin_5.0x3.2mm, symbol Device:Crystal
- R1, R2, R9: footprint jlywxy:0603 -> jlywxy:0402
- R10, R11: value 1.5k -> 5.1k; footprint jlywxy:0603 -> jlywxy:0402
Connections:
- net 1v8_CPUMEM: now also R10.2
- net 1v8_DDR: now also R12.2, R15.2
- net 3v3: now also C28.2, J2.2 (Pin_2), J4.6, R13.2, R22.2, R23.2, R24.2, U4.4 (VDD); no longer R10.2, R12.2, R15.2
- net DEBUG_RXD: now also J2.3 (Pin_3)
- net DEBUG_TXD: now also J2.4 (Pin_4)
- net GND: now also U1.D7 (JTAGSEL), C28.1, J2.1 (Pin_1), J4.7, SW1.1, SW1.2, U4.0 (SHIELD), U4.6 (VSS)
- net JTAG_RST: now also J4.3, R23.1
- net JTAG_TCK: now also J4.5, R24.1
- net JTAG_TDI: now also J4.1, R13.1
- net JTAG_TDO: now also J4.4
- net JTAG_TMS: now also J4.2, R22.1
- net XTAL_IN: now also Y1.2
- net XTAL_OUT: now also Y1.1
- net at C41.2, R11.2, U1.P10 (NRST): now also SW1.3 (K), SW1.4 (A)
- net MCI0_CDA: now reaches U1.P5 (PA16)
- net MCI0_CDA: now also U4.3 (CMD)
- net MCI0_CK: now reaches U1.R5 (PA17)
- net MCI0_CK: now also U4.5 (CLK)
- net MCI0_DA2: now reaches U1.T5 (PA19)
- net MCI0_DA2: now also U4.1 (DAT2)
- net MCI0_DA0: now reaches U1.U4 (PA15)
- net MCI0_DA0: now also U4.7 (DAT0)
- net MCI0_DA1: now reaches U1.U5 (PA18)
- net MCI0_DA1: now also U4.8 (DAT1)
- net MCI0_DA3: now reaches U1.U6 (PA20)
- net MCI0_DA3: now also U4.2 (CD/DAT3)
- net DDR_CLK renamed DDR_CLKP
- net DDR_NCLK renamed DDR_CLKN
- net UART_RXD: no longer names the net of U1.P1 (PA1)
- net UART_TXD: no longer names the net of U1.L3 (PA0)
- net UART_URXD: no longer names the net of U1.G3 (PC9)
- net UART_UTXD renamed SD_DET
- net SD_DET: now also U4.CD
- no-connect marks 116 -> 114
Other:
- note added: "NWAIT"
- moved on the sheet: C41
