File: board/carambola/slimarm_carambola/slimarm_carambola/slimarm_carambola_nonand/slimarm_carambola.kicad_sch (KiCad schematic)
At the start: 69 parts, among them J1 USB_C_Receptacle_USB2.0, J2 Conn_01x04, J4 DF13A-7P-1.25H21, SW1 SW_MEC_5E, U1 AT91SAM9G25-CU, U2 16bit-DDR2-8bank-FBGA84, U3 W25Q128JVS, U5 XC6206PxxxMR, U6 XC6206PxxxMR, U7 XC6206PxxxMR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

Commit message: 23x20f
Parts:
- removed C35, C36: 22pF, jlywxy:0402, symbol Device:C
- removed R12: 470k, jlywxy:0603, symbol Device:R
- removed U6: XC6206PxxxMR, Package_TO_SOT_SMD:SOT-23-3, symbol Regulator_Linear:XC6206PxxxMR
- added C17: 22pF, jlywxy:0402, symbol Device:C
- U5: value XC6206PxxxMR -> AMS1117; footprint Package_TO_SOT_SMD:SOT-23-3 -> Package_TO_SOT_SMD:SOT-89-3
- U7, U8: footprint Package_TO_SOT_SMD:SOT-23-3 -> Package_TO_SOT_SMD:SOT-89-3
Connections:
- net 1v8_DDR: now also C10.2, C11.2, C9.2, U1.D10 (VDDIOM), U1.D13 (VDDIOM), U1.F14 (VDDIOM), C17.2
- net 3v3: now also R10.2
- net at C26.2, R14.2, R15.1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: now also C17.1
- removed net 1v8_CPUMEM: C10.2, C11.2, C9.2, R10.2, U1.D10 (VDDIOM), U1.D13 (VDDIOM), U1.F14 (VDDIOM)
