File: board/slimarm_carambola/pcb_slimarm_carambola-r/slimarm_carambola.kicad_pcb (KiCad board)
At the start: 4 copper layers, 50 x 29.7 mm, 77 parts, among them J1 USB_C_Receptacle_USB2.0, J3 Micro_SD_Card_Det2, J4 DF13A-7P-1.25H21, J5 Conn_01x03, U1 AT91SAM9G25-CU, U2 16bit-DDR2-8bank-FBGA84, U3 SY8089AAAC, U5 AMS1117, U7 XC6206PxxxMR, Y1 Crystal

Commit message: 23x2c7
Parts:
- added J2: Conn_01x14_Pin, Connector_PinHeader_1.27mm:PinHeader_2x07_P1.27mm_Vertical_SMD, B.Cu at (34.3, 38.8)
- added R16: 10k, jlywxy:0402, F.Cu at (26.1, 22.1)
- added R17: 10k, jlywxy:0402, F.Cu at (27.2, 23.7)
- added R18: 10k, jlywxy:0402, F.Cu at (28.9, 21.9)
- added R19: 10k, jlywxy:0402, F.Cu at (27.8, 20.4)
- added R25: 10k, jlywxy:0402, F.Cu at (28.1, 22.8)
- added R26: 39, jlywxy:0603, F.Cu at (41.9, 40.0)
- added R27: 39, jlywxy:0603, F.Cu at (41.8, 38.0)
- moved R12 2.46 mm to (29.8, 21.0), turned to 135 degrees
- moved C2 0.59 mm to (33.5, 17.2)
- moved C5 0.48 mm to (32.6, 18.2)
- moved C1 0.37 mm to (31.6, 19.2)
- moved C3 0.30 mm to (30.7, 20.1)
- moved C28 0.16 mm to (25.4, 25.4)
- moved C8 0.11 mm to (26.3, 24.5)
Connections:
- U1 pad L17: unconnected-(U1C-HFSDPC-PadL17) -> /USB2_DP
- U1 pad M17: unconnected-(U1C-HFSDMC-PadM17) -> /USB2_DN
- U1 pad P16: unconnected-(U1C-HFSDMB-PadP16) -> Net-(U1C-HFSDMB)
- U1 pad P17: unconnected-(U1C-HHSDMB-PadP17) -> /USB1_DN
- U1 pad R16: unconnected-(U1C-HFSDPB-PadR16) -> Net-(U1C-HFSDPB)
- U1 pad R17: unconnected-(U1C-HHSDPB-PadR17) -> /USB1_DP
Routing:
- net /USB2_DN: track 0.00 -> 22.4 mm, vias 0 -> 1
- net /USB2_DP: track 0.00 -> 22.4 mm, vias 0 -> 1
- net /USB1_DP: track 0.00 -> 22.2 mm, vias 0 -> 2
- net /USB1_DN: track 0.00 -> 18.3 mm, vias 0 -> 2
- net /3v3: track 156.1 -> 169.4 mm, vias 20 -> 19
- net /MCI0_DA3: track 20.6 -> 32.9 mm
- net /MCI0_DA2: track 19.5 -> 30.0 mm
- net Net-(U1C-HFSDPB): track 0.00 -> 9.91 mm, vias 0 -> 2
- net Net-(U1C-HFSDMB): track 0.00 -> 9.85 mm, vias 0 -> 2
- net /MCI0_DA1: track 24.9 -> 34.0 mm
- net GND: track 143.6 -> 151.4 mm, vias 49 -> 44
- net /MCI0_DA0: track 20.5 -> 25.8 mm
- net /MCI0_CDA: track 17.9 -> 22.6 mm
- net +5V: track 49.5 -> 51.8 mm
- net Net-(U1C-NRST): track 18.3 -> 16.4 mm
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Other:
- board text added: "Carambola-R v1r1x2c7 AT91SAM9G25@400MHz github: jlywxy/slimarm"
- board text added: "GND RXD TXD"
- board text removed: "Carambola-R v1r0x26b AT91SAM9G25@400MHz github: jlywxy/slimarm"
- board text removed: "G RX TX DBGU"

Commit message: 23x2c7-part2(Carambola)
Routing:
- net /1v8_DDR: track 181.6 -> 180.1 mm
- net Net-(U1C-NRST): track 16.4 -> 17.0 mm

Commit message: 23x2d3
Parts:
- added C36: 100nF, jlywxy:0402, F.Cu at (64.3, 16.2)
- added C39: 100nF, jlywxy:0402, F.Cu at (63.0, 16.2)
- added R28: 5.1k, jlywxy:0402, F.Cu at (47.9, 41.5)
- added U4: MAX811LEUS-T, Package_TO_SOT_SMD:SOT-143, F.Cu at (45.0, 40.5)
- C41: value 22pF -> 100nF
- J2: value Conn_01x14_Pin -> Conn_02x15_Top_Bottom; footprint Connector_PinHeader_1.27mm:PinHeader_2x07_P1.27mm_Vertical_SMD -> Connector_Hirose:Hirose_DF12_DF12E3.0-30DP-0.5V_2x15_P0.50mm_Vertical
- moved C41 31.8 mm to (62.9, 35.9), turned to 90 degrees
- moved R11 16.1 mm to (50.4, 41.5)
- moved J2 0.34 mm to (34.3, 39.1), turned to 0 degrees
Connections:
- C41 pad 2: Net-(U1C-NRST) -> /1v8_DDR
- J2 pad 10: GND -> +5V
- J2 pad 11: GND -> +5V
- J2 pad 12: GND -> +5V
- J2 pad 13: /3v3 -> +5V
- J2 pad 14: GND -> +5V
- J2 pad 2: +5V -> /USB1_DN
- J2 pad 3: /USB1_DN -> /USB1_DP
- J2 pad 4: /USB2_DN -> GND
- J2 pad 5: /USB1_DP -> GND
- J2 pad 6: /USB2_DP -> GND
- J2 pad 7: GND -> /3v3
- J2 pad 8: GND -> /3v3
- J2 pad 9: GND -> +5V
Routing:
- net +5V: track 51.8 -> 67.1 mm, vias 7 -> 9
- net Net-(U1C-NRST): track 17.0 -> 30.4 mm
- net /3v3: track 169.7 -> 180.2 mm, vias 19 -> 24
- net /1v8_DDR: track 180.1 -> 189.3 mm, vias 22 -> 23
- net Net-(U4-~{MR}): track 0.00 -> 4.00 mm
- net /USB2_DP: track 22.4 -> 23.7 mm
- net GND: track 151.5 -> 152.6 mm, vias 44 -> 47
- net /USB1_DP: track 22.2 -> 23.2 mm
Other:
- board text added: "Carambola-R v1r1x2d1 AT91SAM9G25@400MHz github: jlywxy/slimarm"
- board text added: "SlimARM ExtIO"
- board text removed: "Carambola-R v1r1x2c7 AT91SAM9G25@400MHz github: jlywxy/slimarm"
