File: board/slimarm_carambola/pcb_slimarm_carambola-r/slimarm_carambola.kicad_sch (KiCad schematic)
At the start: 72 parts, among them J1 USB_C_Receptacle_USB2.0, J3 Micro_SD_Card_Det2, J4 DF13A-7P-1.25H21, J5 Conn_01x03, U1 AT91SAM9G25-CU, U2 16bit-DDR2-8bank-FBGA84, U3 SY8089AAAC, U5 AMS1117, U7 XC6206PxxxMR, Y1 Crystal

Commit message: 23x2c7
Parts:
- added J2: Conn_01x14_Pin, Connector_PinHeader_1.27mm:PinHeader_2x07_P1.27mm_Vertical_SMD, symbol Connector:Conn_01x14_Pin
- added R16, R17, R18, R19, R25: 10k, jlywxy:0402, symbol Device:R
- added R26, R27: 39, jlywxy:0603, symbol Device:R
Connections:
- net +5V: now also J2.2 (Pin_2)
- net 3v3: now also J2.13 (Pin_13), R16.2, R17.2, R18.2, R19.2, R25.2
- net GND: now also J2.1 (Pin_1), J2.10 (Pin_10), J2.11 (Pin_11), J2.12 (Pin_12), J2.14 (Pin_14), J2.7 (Pin_7), J2.8 (Pin_8), J2.9 (Pin_9)
- net MCI0_CDA: now also R25.1
- net MCI0_DA0: now also R17.1
- net MCI0_DA1: now also R16.1
- net MCI0_DA2: now also R19.1
- net MCI0_DA3: now also R18.1
- net USB2_DP: now reaches U1.L17 (HFSDPC)
- net USB2_DP: now also J2.6 (Pin_6)
- net USB2_DN: now reaches U1.M17 (HFSDMC)
- net USB2_DN: now also J2.4 (Pin_4)
- net at U1.P16 (HFSDMB): now also R27.1
- net USB1_DN: now reaches U1.P17 (HHSDMB)
- net USB1_DN: now also J2.3 (Pin_3), R27.2
- net at U1.R16 (HFSDPB): now also R26.1
- net USB1_DP: now reaches U1.R17 (HHSDPB)
- net USB1_DP: now also J2.5 (Pin_5), R26.2
- no-connect marks 107 -> 99
Other:
- note added: "SlimARM Carambola v1r1 APPROVAL this version: 1. fixed SDIO pull-up 2. added extension IO"

Commit message: 23x2c7-part2(Carambola)
Connections:
- no-connect marks 99 -> 105
Changed lines of the file:
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@@
   (no_connect (at 287.02 69.85))
   (no_connect (at 25.4 36.83))
+  (no_connect (at 134.62 96.52))
   (no_connect (at 25.4 105.41))
   (no_connect (at 96.52 118.11))
@@
   (no_connect (at 96.52 36.83))
   (no_connect (at 134.62 63.5))
+  (no_connect (at 134.62 93.98))
   (no_connect (at 101.6 195.58))
   (no_connect (at 134.62 50.8))
@@
   (no_connect (at 25.4 110.49))
   (no_connect (at 101.6 215.9))
+  (no_connect (at 134.62 43.18))
   (no_connect (at 101.6 205.74))
   (no_connect (at 101.6 223.52))
@@
   (no_connect (at 25.4 77.47))
   (no_connect (at 96.52 74.93))
+  (no_connect (at 96.52 41.91))
   (no_connect (at 96.52 46.99))
   (no_connect (at 25.4 123.19))
@@
   (no_connect (at 96.52 95.25))
   (no_connect (at 25.4 220.98))
+  (no_connect (at 134.62 99.06))
+  (no_connect (at 134.62 114.3))
   (no_connect (at 25.4 39.37))
   (no_connect (at 134.62 106.68))
@@
     (stroke (width 0) (type default))
   )
+  (wire (pts (xy 198.12 203.2) (xy 195.58 203.2))
+    (stroke (width 0) (type default))
+  )
   (wire (pts (xy 111.76 203.2) (xy 118.11 203.2))
     (stroke (width 0) (type default))
@@
     )
   )
-  (symbol (lib_id "power:GND") (at 195.58 203.2 90) (unit 1)
+  (symbol (lib_id "power:GND") (at 198.12 203.2 90) (unit 1)
     (in_bom yes) (on_board yes) (dnp no) (fields_autoplaced)
-    (property "Reference" "#PWR047" (at 201.93 203.2 0)
+    (property "Reference" "#PWR047" (at 204.47 203.2 0)
       (effects (font (size 1.27 1.27)) hide)
     )
-    (property "Value" "GND" (at 199.39 203.835 90)
+    (property "Value" "GND" (at 201.93 203.835 90)
       (effects (font (size 1.27 1.27)) (justify right))
     )
-    (property "Footprint" "" (at 195.58 203.2 0)
+    (property "Footprint" "" (at 198.12 203.2 0)
       (effects (font (size 1.27 1.27)) hide)
     )
-    (property "Datasheet" "" (at 195.58 203.2 0)
+    (property "Datasheet" "" (at 198.12 203.2 0)
       (effects (font (size 1.27 1.27)) hide)
     )

Commit message: 23x2d3
Parts:
- removed J2: Conn_01x14_Pin, Connector_PinHeader_1.27mm:PinHeader_2x07_P1.27mm_Vertical_SMD, symbol Connector:Conn_01x14_Pin
- added C36, C39: 100nF, jlywxy:0402, symbol Device:C
- added J2: Conn_02x15_Top_Bottom, Connector_Hirose:Hirose_DF12_DF12E3.0-30DP-0.5V_2x15_P0.50mm_Vertical, symbol Connector_Generic:Conn_02x15_Top_Bottom
- added R28: 5.1k, jlywxy:0402, symbol Device:R
- added U4: MAX811LEUS-T, Package_TO_SOT_SMD:SOT-143, symbol Power_Supervisor:MAX811LEUS-T
- C41: value 22pF -> 100nF
Connections:
- net +5V: now also J2.10 (Pin_10), J2.11 (Pin_11), J2.12 (Pin_12), J2.13 (Pin_13), J2.14 (Pin_14), J2.15 (Pin_15), J2.9 (Pin_9)
- net 1v8_DDR: now also C41.2, C36.2, C39.2
- net 3v3: now also J2.7 (Pin_7), J2.8 (Pin_8), R28.1, U4.4 (VCC)
- net GND: now also C36.1, C39.1, J2.1 (Pin_1), J2.16 (Pin_16), J2.19 (Pin_19), J2.20 (Pin_20), J2.21 (Pin_21), J2.22 (Pin_22), J2.23 (Pin_23), J2.24 (Pin_24), J2.25 (Pin_25), J2.26 (Pin_26), J2.27 (Pin_27), J2.28 (Pin_28), J2.29 (Pin_29), J2.30 (Pin_30), J2.4 (Pin_4), J2.5 (Pin_5), J2.6 (Pin_6), U4.1 (GND)
- net USB1_DN: now also J2.2 (Pin_2)
- net USB1_DP: now also J2.3 (Pin_3)
- net USB2_DN: now also J2.17 (Pin_17)
- net USB2_DP: now also J2.18 (Pin_18)
- net at R11.2, U1.P10 (NRST): now also U4.2 (~{RESET}); no longer C41.2
- new net: R28.2, U4.3 (~{MR})
