File: board/slimarm_hypericum/pcb_slimarm_hypericum_d/slimarm_hypericum.kicad_pcb (KiCad board)
At the start: 4 copper layers, 50 x 33.5 mm, 131 parts, among them J1 USB_C_Receptacle_USB2.0, J2 Micro_SD_Card_Det2, J3 Conn_01x03, J4 Conn_01x14_Pin, J5 DF13A-7P-1.25H21, U1 AllWinner-A20, U2 K4B8G1646B-MCK0, U3 SY8089AAAC, U4 SY8089AAAC, U5 SY8089AAAC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

Commit message: 23x2d3
Parts:
- removed C18, C58, C59: 100nF, jlywxy:0402
- removed J4: Conn_01x14_Pin, Connector_PinHeader_1.27mm:PinHeader_2x07_P1.27mm_Vertical_SMD
- added J6: Conn_02x15_Top_Bottom, Connector_Hirose:Hirose_DF12_DF12C3.0-30DS-0.5V_2x15_P0.50mm_Vertical, B.Cu at (40.6, 102.9)
- added R32: 5.1k, jlywxy:0402, F.Cu at (68.0, 75.8)
- added U9: MAX811LEUS-T, Package_TO_SOT_SMD:SOT-143, F.Cu at (53.4, 74.8)
- moved R20 6.57 mm to (45.7, 78.4), turned to 0 degrees
- moved R25 4.49 mm to (48.6, 76.6), turned to 180 degrees
- moved R26 2.93 mm to (45.7, 77.2), turned to 0 degrees
- moved R5 0.52 mm to (55.8, 74.7)
- moved C74 0.44 mm to (62.9, 74.2)
- moved C81 0.44 mm to (57.1, 74.3)
- moved R17 0.44 mm to (58.5, 74.6)
- moved C37 0.44 mm to (68.6, 74.2)
- moved C75 0.44 mm to (67.3, 74.2)
- moved C82 0.44 mm to (61.5, 74.2)
- moved R15 0.44 mm to (64.3, 74.6)
- moved R16 0.44 mm to (65.9, 74.6)
- moved R18 0.44 mm to (60.1, 74.6)
Connections:
- R25 pad 1: +3V3 -> Net-(U1D-RESET#)
- R25 pad 2: Net-(U1D-RESET#) -> +3V3
Routing:
- net +3V3: track 209.5 -> 247.5 mm, vias 20 -> 22
- net Net-(U9-~{MR}): track 0.00 -> 15.0 mm, vias 0 -> 2
- net GND: track 263.0 -> 274.5 mm, vias 76 -> 72
- net +5V: track 136.5 -> 147.2 mm, vias 12 -> 13
- net /USB_DN2: track 22.5 -> 30.6 mm
- net /USB_DP2: track 21.9 -> 27.9 mm
- net +2V5: track 34.8 -> 38.4 mm, vias 5 -> 7
- net Net-(U1D-RESET#): track 40.5 -> 43.8 mm
- net /SD1_CLK: track 11.5 -> 14.7 mm, vias 1 -> 2
- net /SD1_DAT3: track 8.65 -> 11.7 mm, vias 1 -> 2
- net /SD1_DAT1: track 10.00 -> 12.9 mm, vias 1 -> 2
- net +1V5: track 230.7 -> 228.4 mm, vias 26 -> 25
- net Net-(U1D-JTAGSEL): track 17.3 -> 15.2 mm
- net Net-(U1D-BOOTSEL): track 17.0 -> 15.0 mm
- net /SD1_DAT2: track 14.5 -> 16.4 mm, vias 1 -> 2
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Other:
- board text added: "Hypericum-R v1r1x2d1 Allwinner-A20@1.2GHz github: jlywxy/slimarm"
- board text added: "SlimARM ExtIO"
- board text removed: "GND 5v DN1 DN2 DP1 DP2 D3 D2 D1 D0 CLK CMD 3v3 GND"
- board text removed: "Hypericum-R v1r0x2bf Allwinner-A20@1.2GHz github: jlywxy/slimarm"
