File: board/slimarm_hypericum/pcb_slimarm_hypericum_d/slimarm_hypericum.kicad_sch (KiCad schematic)
At the start: 127 parts, among them J1 USB_C_Receptacle_USB2.0, J2 Micro_SD_Card_Det2, J3 Conn_01x03, J4 Conn_01x14_Pin, J5 DF13A-7P-1.25H21, U1 AllWinner-A20, U2 K4B8G1646B-MCK0, U3 SY8089AAAC, U4 SY8089AAAC, U5 SY8089AAAC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

Commit message: 23x2d3
Parts:
- removed C18, C58, C59: 100nF, jlywxy:0402, symbol Device:C
- removed J4: Conn_01x14_Pin, Connector_PinHeader_1.27mm:PinHeader_2x07_P1.27mm_Vertical_SMD, symbol Connector:Conn_01x14_Pin
- added J6: Conn_02x15_Top_Bottom, Connector_Hirose:Hirose_DF12_DF12C3.0-30DS-0.5V_2x15_P0.50mm_Vertical, symbol Connector_Generic:Conn_02x15_Top_Bottom
- added R32: 5.1k, jlywxy:0402, symbol Device:R
- added U9: MAX811LEUS-T, Package_TO_SOT_SMD:SOT-143, symbol Power_Supervisor:MAX811LEUS-T
Connections:
- net +3V3: now also R25.2, J6.7 (Pin_7), J6.8 (Pin_8), R32.1, U9.4 (VCC); no longer R25.1
- net +5V: now also J6.10 (Pin_10), J6.11 (Pin_11), J6.12 (Pin_12), J6.13 (Pin_13), J6.14 (Pin_14), J6.15 (Pin_15), J6.9 (Pin_9)
- net GND: now also J6.1 (Pin_1), J6.16 (Pin_16), J6.25 (Pin_25), J6.26 (Pin_26), J6.27 (Pin_27), J6.28 (Pin_28), J6.29 (Pin_29), J6.30 (Pin_30), J6.4 (Pin_4), J6.5 (Pin_5), J6.6 (Pin_6), U9.1 (GND)
- net SD1_CLK: now also J6.19 (Pin_19)
- net SD1_CMD: now also J6.20 (Pin_20)
- net SD1_DAT0: now also J6.21 (Pin_21)
- net SD1_DAT1: now also J6.22 (Pin_22)
- net SD1_DAT2: now also J6.23 (Pin_23)
- net SD1_DAT3: now also J6.24 (Pin_24)
- net USB_DN1: now also J6.2 (Pin_2)
- net USB_DN2: now also J6.17 (Pin_17)
- net USB_DP1: now also J6.3 (Pin_3)
- net USB_DP2: now also J6.18 (Pin_18)
- net at U1.C14 (RESET#): now also R25.1, U9.2 (~{RESET}); no longer R25.2
- new net: R32.2, U9.3 (~{MR})
Other:
- note added: "Hypericum Release v1r1 APPROVAL 2023.7.21 1. applied extension interface "SlimARM ExtIO" 2. use reset chip for cpu reset"
